File: V5/Main-v5.1.brd (EAGLE design)
At the start: 80 x 80 mm, 111 parts, among them IC1 MC34063AD, J11 AVR_SPI_PROG_3X2NS, M01 JUMPER-SMT_2_NC_PASTE_SILK, M02 JUMPER-SMT_2_NC_PASTE_SILK, M11 JUMPER-SMT_2_NC_PASTE_SILK, M12 JUMPER-SMT_2_NC_PASTE_SILK, Q1 MOSFET-NCHANNEL2N7002PW, Q2 MOSFET-NCHANNEL2N7002PW, U1 ULN2803ADWG4, U10 FSMSMTR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

Commit message: Added SPI connector for SD card and modified UART programmer to support ATmega in V5.1
Parts:
- added C20: 0.1uf, resistor:C0603
- added J7: (no value), SparkFun-Connectors:1X06
- added J8: (no value), SparkFun-Connectors:1X02
- added JP4, JP5: JUMPER-SMT_3_2-NC_PASTE_SILK, SparkFun-Jumpers:SMT-JUMPER_3_2-NC_PASTE_SILK
- moved U10 5.43 mm to (12.7, 7.94)
- moved J11 5.24 mm to (19.1, 11.4)
- moved LED6 4.86 mm to (18.1, 18.7)
- moved R25 4.80 mm to (20.3, 18.7)
- moved JP1 4.49 mm to (45.4, 40.6)
- moved JP2 4.49 mm to (48.6, 40.6)
- moved R13 1.90 mm to (8.89, 66.7)
- moved R24 1.59 mm to (7.62, 13.0)
Connections:
- removed net RGB-3: U7.14
- new net N$72: J10.4, JP4.2
- new net N$81: J10.5, JP5.2
- new net SS_SD: J7.6, U7.14
- new net VCC_FTDI: J10.3
- net +3V3: no longer J10.3
- net +5V: now also J7.2
- net DTR: now also C20.1
- net ESPRX: now also JP4.1; no longer J10.4
- net ESPTX: now also JP5.1; no longer J10.5
- net GND: now also J7.1, J8.1
- net MEGARX: now also JP4.3
- net MEGATX: now also JP5.3
- net MISO: now also J7.3
- net MOSI: now also J7.4
- net RST: now also C20.2
- net SCK: now also J7.5
- net VCC: now also J8.2
Routing:
- net VCC: track 143.1 -> 191.2 mm
- net N$72: track 0.00 -> 44.4 mm, vias 0 -> 1
- net N$81: track 0.00 -> 42.9 mm, vias 0 -> 1
- net RST: track 55.5 -> 93.5 mm, vias 2 -> 8
- net MEGATX: track 17.5 -> 44.7 mm, vias 2 -> 3
- net SS_SD: track 0.00 -> 20.4 mm
- net MEGARX: track 17.6 -> 35.8 mm, vias 2 -> 3
- net MISO: track 23.3 -> 41.3 mm, vias 1 -> 3
- net GND: track 371.8 -> 358.8 mm, vias 29 -> 31
- net ESPRX: track 42.4 -> 30.4 mm
- net +3V3: track 166.3 -> 156.1 mm
- net +5V: track 284.8 -> 293.8 mm, vias 16 -> 15
- net SCK: track 23.5 -> 32.3 mm
- net ESPTX: track 44.5 -> 37.7 mm
- net N$57: track 14.8 -> 20.9 mm, vias 2 -> 0
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