File: V5/Main-v5.1.sch (EAGLE design)
At the start: 109 parts, among them IC1 MC34063AD, J11 AVR_SPI_PROG_3X2NS, M01 JUMPER-SMT_2_NC_PASTE_SILK, M02 JUMPER-SMT_2_NC_PASTE_SILK, M11 JUMPER-SMT_2_NC_PASTE_SILK, M12 JUMPER-SMT_2_NC_PASTE_SILK, Q1 MOSFET-NCHANNEL2N7002PW, Q2 MOSFET-NCHANNEL2N7002PW, U1 ULN2803ADWG4, U10 FSMSMTR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

Commit message: Added SPI connector for SD card and modified UART programmer to support ATmega in V5.1
Parts:
- added C20: 0.1uf, resistor:C-EUC0603
- added J7: (no value), SparkFun-Connectors:CONN_06SILK_FEMALE_PTH
- added J8: (no value), SparkFun-Connectors:CONN_02
- added JP4, JP5: JUMPER-SMT_3_2-NC_PASTE_SILK, SparkFun-Jumpers:JUMPER-SMT_3_2-NC_PASTE_SILK
Connections:
- removed net RGB-3: U7.PB2(SS/OC1B)
- new net N$72: J10.4, JP4.2
- new net N$81: J10.5, JP5.2
- new net SS_SD: J7.6, U7.PB2(SS/OC1B)
- new net VCC_FTDI: J10.3
- net +3V3: no longer J10.3
- net +5V: now also J7.2
- net DTR: now also C20.1
- net ESPRX: now also JP4.1; no longer J10.4
- net ESPTX: now also JP5.1; no longer J10.5
- net GND: now also J7.1, J8.1
- net MEGARX: now also JP4.3
- net MEGATX: now also JP5.3
- net MISO: now also J7.3
- net MOSI: now also J7.4
- net RST: now also C20.2
- net SCK: now also J7.5
- net VCC: now also J8.2
Other:
- moved on the sheet: J10
