File: V6/Main-v6.0 copy.brd (EAGLE design)
At the start: 80 x 80 mm, 106 parts, among them J11 AVR_SPI_PROG_3X2NS, M01 JUMPER-SMT_2_NC_PASTE_SILK, M02 JUMPER-SMT_2_NC_PASTE_SILK, M11 JUMPER-SMT_2_NC_PASTE_SILK, M12 JUMPER-SMT_2_NC_PASTE_SILK, Q1 MOSFET-NCHANNEL2N7002PW, Q2 MOSFET-NCHANNEL2N7002PW, U1 ULN2803ADWG4, U10 FSMSMTR, U2 ULN2803ADWG4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

Commit message: V6.0 Copy Routed Board
Parts:
- moved C10 1.27 mm to (21.6, 33.0)
- moved C9 1.06 mm to (21.0, 29.4)
- moved R18 0.90 mm to (21.1, 27.9)
- moved C11 0.63 mm to (20.3, 55.2)
- moved R3 0.63 mm to (9.19, 49.0)
- moved R6 0.63 mm to (10.5, 49.0)
- moved R8 0.63 mm to (20.3, 54.0)
- turned LED5 to 0 degrees
- turned LED6 to 180 degrees
Routing:
- net +5V: track 0.00 -> 267.6 mm, vias 0 -> 11
- net VCC: track 0.00 -> 163.4 mm, vias 0 -> 7
- net +3V3: track 0.00 -> 138.7 mm, vias 0 -> 8
- net RST: track 0.00 -> 109.8 mm, vias 0 -> 2
- net N$72: track 0.00 -> 97.6 mm, vias 0 -> 6
- net PULSE: track 0.00 -> 88.6 mm, vias 0 -> 3
- net +24V: track 0.00 -> 76.3 mm, vias 0 -> 2
- net GPIO0: track 0.00 -> 56.0 mm, vias 0 -> 2
- net STEP2: track 0.00 -> 55.0 mm, vias 0 -> 2
- net A0: track 0.00 -> 49.5 mm, vias 0 -> 2
- net N$81: track 0.00 -> 47.9 mm, vias 0 -> 3
- net A1: track 0.00 -> 46.5 mm, vias 0 -> 2
- net MEGATX: track 0.00 -> 38.6 mm, vias 0 -> 2
- net ENB: track 0.00 -> 38.3 mm, vias 0 -> 2
- net DIR2: track 0.00 -> 37.9 mm, vias 0 -> 2
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